File: examples/stm32_usb_buck/stm32/stm32.sch (KiCad schematic (older format))
At the start: 3 parts, among them U1 STM32F405RGTx

Commit message: adding schematic
Parts:
- added C3: (no value), symbol Device:C
- added D1, D2: (no value), symbol Device:D
- added R1, R2, R3, R4: (no value), symbol Device:R
- added U2: (no value), symbol 74xGxx:74LVC1G66
- C1, C2: value C_Small -> (none)
- U1: value STM32F405RGTx -> (none); footprint Package_QFP:LQFP-64_10x10mm_P0.5mm -> (none)
Connections:
- wire segments 0 -> 8
Changed lines of the file:
@@
 $Comp
 L MCU_ST_STM32F4:STM32F405RGTx U1
-U 1 1 6111500c
-P 4000 2500
-F 0 "U1" H 3400 4250 50 000 L CNN
-F 1 "STM32F405RGTx" H 4400 4250 50 000 L CNN
-F 2 "Package_QFP:LQFP-64_10x10mm_P0.5mm" H 3400 800 50 000 C CNN
-F 3 "" H 4000 2500 50 000 C CNN
-   1   4000 2500
+U 1 1 6114aeca
+P 16550 11650
+F 0 "U1" H 15950 13400 50 000 L CNN
+   1   16550 11650
    1   0  0  -1
 $EndComp
 $Comp
 L Device:C_Small C1
-U 1 1 6111500c
-P 3000 1600
-F 0 "C1" H 3010 1670 50 000 L CNN
-F 1 "C_Small" H 3010 1520 50 000 L CNN
-F 2 "" H 3000 1600 50 000 C CNN
-F 3 "" H 3000 1600 50 000 C CNN
-   1   3000 1600
+U 1 1 6114aeca
+P 15650 10550
+F 0 "C1" H 15660 10620 50 000 L CNN
+   1   15650 10550
    1   0  0  -1
 $EndComp
 $Comp
 L Device:C_Small C2
-U 1 1 6111500c
-P 3100 1500
-F 0 "C2" H 3110 1570 50 000 L CNN
-F 1 "C_Small" H 3110 1420 50 000 L CNN
-F 2 "" H 3100 1500 50 000 C CNN
-F 3 "" H 3100 1500 50 000 C CNN
-   1   3100 1500
+U 1 1 6114aeca
+P 15450 10650
+F 0 "C2" H 15460 10720 50 000 L CNN
+   1   15450 10650
    1   0  0  -1
 $EndComp
+$Comp
+L Device:D D1
+U 1 1 6114aeca
+P 17750 11850
+F 0 "D1" H 17750 11950 50 000 C CNN
+   1   17750 11850
+   1   0  0  -1
+$EndComp
+$Comp
+L Device:R R1
+U 1 1 6114aeca
+P 17450 11700
+F 0 "R1" V 17530 11700 50 000 C CNN
+   1   17450 11700
+   1   0  0  -1
+$EndComp
+$Comp
+L 74xGxx:74LVC1G66 U2
+U 1 1 6114aeca
+P 18550 13650
+F 0 "U2" H 18450 13850 50 000 C CNN
+   1   18550 13650
+   1   0  0  -1
+$EndComp
+$Comp
+L Device:R R2
+U 1 1 6114aeca
+P 17900 13800
+F 0 "R2" V 17980 13800 50 000 C CNN
+   1   17900 13800
+   1   0  0  -1
+$EndComp
+$Comp
+L Device:R R3
+U 1 1 6114aeca
+P 19000 13800
+F 0 "R3" V 19080 13800 50 000 C CNN
+   1   19000 13800
+   1   0  0  -1
+$EndComp
+$Comp
+L Device:C C3
+U 1 1 6114aeca
+P 18550 13250
+F 0 "C3" H 18575 13350 50 000 L CNN
+   1   18550 13250
+   1   0  0  -1
+$EndComp
+$Comp
+L Device:D D2
+U 1 1 6114aeca
+P 18250 13800
+F 0 "D2" H 18250 13900 50 000 C CNN
+   1   18250 13800
+   1   0  0  -1
+$EndComp
+$Comp
+L Device:R R4
+U 1 1 6114aeca
+P 18550 13650
+F 0 "R4" V 18630 13650 50 000 C CNN
+   1   18550 13650
+   1   0  0  -1
+$EndComp
+Wire Wire Line
+	15650 10450 15850 10450
+Wire Wire Line
+	19000 13650 18800 13650
+Wire Wire Line
+	18400 13800 18300 13800
+Wire Wire Line
+	18100 13800 18550 13800
+Wire Wire Line
+	17450 11550 17250 11550
+Wire Wire Line
+	17900 13650 18300 13650
+Wire Wire Line
+	17600 11850 17450 11850
+Wire Wire Line
+	15450 10550 15850 10550
 $EndSCHEMATC

Commit message: Changed 'sch_loc' to 'sch_bb' and added 2 fields for height and width.  Changed gen_bbox to be a Part method that acts on iteself
Changed lines of the file:
@@
 $Comp
 L MCU_ST_STM32F4:STM32F405RGTx U1
-U 1 1 6114aeca
+U 1 1 611815fd
 P 16550 11650
 F 0 "U1" H 15950 13400 50 000 L CNN
@@
 $Comp
 L Device:C_Small C1
-U 1 1 6114aeca
-P 15650 10550
-F 0 "C1" H 15660 10620 50 000 L CNN
-   1   15650 10550
+U 1 1 611815fd
+P 15450 10550
+F 0 "C1" H 15460 10620 50 000 L CNN
+   1   15450 10550
    1   0  0  -1
 $EndComp
 $Comp
 L Device:C_Small C2
-U 1 1 6114aeca
-P 15450 10650
-F 0 "C2" H 15460 10720 50 000 L CNN
-   1   15450 10650
+U 1 1 611815fd
+P 15650 10650
+F 0 "C2" H 15660 10720 50 000 L CNN
+   1   15650 10650
    1   0  0  -1
 $EndComp
 $Comp
 L Device:D D1
-U 1 1 6114aeca
-P 17750 11850
-F 0 "D1" H 17750 11950 50 000 C CNN
-   1   17750 11850
+U 1 1 611815fd
+P 16550 11650
+F 0 "D1" H 16550 11750 50 000 C CNN
+   1   16550 11650
    1   0  0  -1
 $EndComp
 $Comp
 L Device:R R1
-U 1 1 6114aeca
+U 1 1 611815fd
 P 17450 11700
 F 0 "R1" V 17530 11700 50 000 C CNN
@@
 $Comp
 L 74xGxx:74LVC1G66 U2
-U 1 1 6114aeca
+U 1 1 611815fd
 P 18550 13650
 F 0 "U2" H 18450 13850 50 000 C CNN
@@
 $Comp
 L Device:R R2
-U 1 1 6114aeca
+U 1 1 611815fd
 P 17900 13800
 F 0 "R2" V 17980 13800 50 000 C CNN
@@
 $Comp
 L Device:R R3
-U 1 1 6114aeca
+U 1 1 611815fd
 P 19000 13800
 F 0 "R3" V 19080 13800 50 000 C CNN
@@
 $Comp
 L Device:C C3
-U 1 1 6114aeca
+U 1 1 611815fd
 P 18550 13250
 F 0 "C3" H 18575 13350 50 000 L CNN
@@
 $Comp
 L Device:D D2
-U 1 1 6114aeca
+U 1 1 611815fd
 P 18250 13800
 F 0 "D2" H 18250 13900 50 000 C CNN
@@
 $Comp
 L Device:R R4
-U 1 1 6114aeca
+U 1 1 611815fd
 P 18550 13650
 F 0 "R4" V 18630 13650 50 000 C CNN
@@
 $EndComp
 Wire Wire Line
-	15650 10450 15850 10450
+	18300 13800 18400 13800
 Wire Wire Line
-	19000 13650 18800 13650
+	18800 13650 19000 13650
 Wire Wire Line
-	18400 13800 18300 13800
+	17250 11550 17450 11550
 Wire Wire Line
-	18100 13800 18550 13800
+	18300 13650 17900 13650
 Wire Wire Line
-	17450 11550 17250 11550
+	18550 13800 18100 13800
 Wire Wire Line
-	17900 13650 18300 13650
+	15850 10550 15650 10550
 Wire Wire Line
-	17600 11850 17450 11850
+	17450 11850 16400 11650
 Wire Wire Line
-	15450 10550 15850 10550
+	15850 10450 15450 10450
 $EndSCHEMATC

Commit message: bounding box collision kinda working
Parts:
- removed C3: (no value), symbol Device:C
- removed D2: (no value), symbol Device:D
- removed R2, R3, R4: (no value), symbol Device:R
- removed U2: (no value), symbol 74xGxx:74LVC1G66
Connections:
- wire segments 8 -> 4
Changed lines of the file:
@@
 $Comp
 L MCU_ST_STM32F4:STM32F405RGTx U1
-U 1 1 611815fd
+U 1 1 61182a18
 P 16550 11650
 F 0 "U1" H 15950 13400 50 000 L CNN
@@
 $Comp
 L Device:C_Small C1
-U 1 1 611815fd
-P 15450 10550
-F 0 "C1" H 15460 10620 50 000 L CNN
-   1   15450 10550
+U 1 1 61182a18
+P 15850 10550
+F 0 "C1" H 15860 10620 50 000 L CNN
+   1   15850 10550
    1   0  0  -1
 $EndComp
 $Comp
 L Device:C_Small C2
-U 1 1 611815fd
-P 15650 10650
-F 0 "C2" H 15660 10720 50 000 L CNN
-   1   15650 10650
+U 1 1 61182a18
+P 15850 10650
+F 0 "C2" H 15860 10720 50 000 L CNN
+   1   15850 10650
    1   0  0  -1
 $EndComp
 $Comp
 L Device:D D1
-U 1 1 611815fd
+U 1 1 61182a18
 P 16550 11650
 F 0 "D1" H 16550 11750 50 000 C CNN
@@
 $Comp
 L Device:R R1
-U 1 1 611815fd
-P 17450 11700
-F 0 "R1" V 17530 11700 50 000 C CNN
-   1   17450 11700
-   1   0  0  -1
-$EndComp
-$Comp
-L 74xGxx:74LVC1G66 U2
-U 1 1 611815fd
-P 18550 13650
-F 0 "U2" H 18450 13850 50 000 C CNN
-   1   18550 13650
-   1   0  0  -1
-$EndComp
-$Comp
-L Device:R R2
-U 1 1 611815fd
-P 17900 13800
-F 0 "R2" V 17980 13800 50 000 C CNN
-   1   17900 13800
-   1   0  0  -1
-$EndComp
-$Comp
-L Device:R R3
-U 1 1 611815fd
-P 19000 13800
-F 0 "R3" V 19080 13800 50 000 C CNN
-   1   19000 13800
-   1   0  0  -1
-$EndComp
-$Comp
-L Device:C C3
-U 1 1 611815fd
-P 18550 13250
-F 0 "C3" H 18575 13350 50 000 L CNN
-   1   18550 13250
-   1   0  0  -1
-$EndComp
-$Comp
-L Device:D D2
-U 1 1 611815fd
-P 18250 13800
-F 0 "D2" H 18250 13900 50 000 C CNN
-   1   18250 13800
-   1   0  0  -1
-$EndComp
-$Comp
-L Device:R R4
-U 1 1 611815fd
-P 18550 13650
-F 0 "R4" V 18630 13650 50 000 C CNN
-   1   18550 13650
+U 1 1 61182a18
+P 17250 11700
+F 0 "R1" V 17330 11700 50 000 C CNN
+   1   17250 11700
    1   0  0  -1
 $EndComp
 Wire Wire Line
-	18300 13800 18400 13800
+	17250 11550 17250 11550
 Wire Wire Line
-	18800 13650 19000 13650
+	17250 11850 16400 11650
 Wire Wire Line
-	17250 11550 17450 11550
+	15850 10550 15850 10550
 Wire Wire Line
-	18300 13650 17900 13650
-Wire Wire Line
-	18550 13800 18100 13800
-Wire Wire Line
-	15850 10550 15650 10550
-Wire Wire Line
-	17450 11850 16400 11650
-Wire Wire Line
-	15850 10450 15450 10450
+	15850 10450 15850 10450
 $EndSCHEMATC

Commit message: basic auto layout working around center part
Changed lines of the file:
@@
 $Comp
 L MCU_ST_STM32F4:STM32F405RGTx U1
-U 1 1 61182a18
+U 1 1 61182d78
 P 16550 11650
 F 0 "U1" H 15950 13400 50 000 L CNN
@@
 $Comp
 L Device:C_Small C1
-U 1 1 61182a18
-P 15850 10550
-F 0 "C1" H 15860 10620 50 000 L CNN
-   1   15850 10550
+U 1 1 61182d78
+P 15350 10550
+F 0 "C1" H 15360 10620 50 000 L CNN
+   1   15350 10550
    1   0  0  -1
 $EndComp
 $Comp
 L Device:C_Small C2
-U 1 1 61182a18
-P 15850 10650
-F 0 "C2" H 15860 10720 50 000 L CNN
-   1   15850 10650
+U 1 1 61182d78
+P 15650 10650
+F 0 "C2" H 15660 10720 50 000 L CNN
+   1   15650 10650
    1   0  0  -1
 $EndComp
 $Comp
 L Device:D D1
-U 1 1 61182a18
+U 1 1 61182d78
 P 16550 11650
 F 0 "D1" H 16550 11750 50 000 C CNN
@@
 $Comp
 L Device:R R1
-U 1 1 61182a18
-P 17250 11700
-F 0 "R1" V 17330 11700 50 000 C CNN
-   1   17250 11700
+U 1 1 61182d78
+P 17450 11700
+F 0 "R1" V 17530 11700 50 000 C CNN
+   1   17450 11700
    1   0  0  -1
 $EndComp
 Wire Wire Line
-	17250 11550 17250 11550
+	17250 11550 17450 11550
 Wire Wire Line
-	17250 11850 16400 11650
+	15850 10550 15650 10550
 Wire Wire Line
-	15850 10550 15850 10550
+	17450 11850 16400 11650
 Wire Wire Line
-	15850 10450 15850 10450
+	15850 10450 15350 10450
 $EndSCHEMATC

Commit message: Auto moving parts in increments of 50
Parts:
- added C3: (no value), symbol Device:C
- added D2: (no value), symbol Device:D
- added R2, R3, R4: (no value), symbol Device:R
- added U2: (no value), symbol 74xGxx:74LVC1G66
Connections:
- wire segments 4 -> 8
Changed lines of the file:
@@
 $Comp
 L MCU_ST_STM32F4:STM32F405RGTx U1
-U 1 1 61182d78
+U 1 1 611830cb
 P 16550 11650
 F 0 "U1" H 15950 13400 50 000 L CNN
@@
 $Comp
 L Device:C_Small C1
-U 1 1 61182d78
-P 15350 10550
-F 0 "C1" H 15360 10620 50 000 L CNN
-   1   15350 10550
+U 1 1 611830cb
+P 15450 10550
+F 0 "C1" H 15460 10620 50 000 L CNN
+   1   15450 10550
    1   0  0  -1
 $EndComp
 $Comp
 L Device:C_Small C2
-U 1 1 61182d78
-P 15650 10650
-F 0 "C2" H 15660 10720 50 000 L CNN
-   1   15650 10650
+U 1 1 611830cb
+P 15700 10650
+F 0 "C2" H 15710 10720 50 000 L CNN
+   1   15700 10650
    1   0  0  -1
 $EndComp
 $Comp
 L Device:D D1
-U 1 1 61182d78
+U 1 1 611830cb
 P 16550 11650
 F 0 "D1" H 16550 11750 50 000 C CNN
@@
 $Comp
 L Device:R R1
-U 1 1 61182d78
-P 17450 11700
-F 0 "R1" V 17530 11700 50 000 C CNN
-   1   17450 11700
+U 1 1 611830cb
+P 17400 11700
+F 0 "R1" V 17480 11700 50 000 C CNN
+   1   17400 11700
+   1   0  0  -1
+$EndComp
+$Comp
+L 74xGxx:74LVC1G66 U2
+U 1 1 611830cb
+P 18550 13650
+F 0 "U2" H 18450 13850 50 000 C CNN
+   1   18550 13650
+   1   0  0  -1
+$EndComp
+$Comp
+L Device:R R2
+U 1 1 611830cb
+P 17800 13800
+F 0 "R2" V 17880 13800 50 000 C CNN
+   1   17800 13800
+   1   0  0  -1
+$EndComp
+$Comp
+L Device:R R3
+U 1 1 611830cb
+P 18950 13800
+F 0 "R3" V 19030 13800 50 000 C CNN
+   1   18950 13800
+   1   0  0  -1
+$EndComp
+$Comp
+L Device:C C3
+U 1 1 611830cb
+P 18550 13250
+F 0 "C3" H 18575 13350 50 000 L CNN
+   1   18550 13250
+   1   0  0  -1
+$EndComp
+$Comp
+L Device:D D2
+U 1 1 611830cb
+P 18100 13800
+F 0 "D2" H 18100 13900 50 000 C CNN
+   1   18100 13800
+   1   0  0  -1
+$EndComp
+$Comp
+L Device:R R4
+U 1 1 611830cb
+P 18550 13650
+F 0 "R4" V 18630 13650 50 000 C CNN
+   1   18550 13650
    1   0  0  -1
 $EndComp
 Wire Wire Line
-	17250 11550 17450 11550
+	18300 13800 18250 13800
 Wire Wire Line
-	15850 10550 15650 10550
+	17400 11850 16400 11650
 Wire Wire Line
-	17450 11850 16400 11650
+	18300 13650 17800 13650
 Wire Wire Line
-	15850 10450 15350 10450
+	18800 13650 18950 13650
+Wire Wire Line
+	15850 10550 15700 10550
+Wire Wire Line
+	18550 13800 17950 13800
+Wire Wire Line
+	15850 10450 15450 10450
+Wire Wire Line
+	17250 11550 17400 11550
 $EndSCHEMATC

Commit message: refactored rectangle code into a function
Changed lines of the file:
@@
 $Comp
 L MCU_ST_STM32F4:STM32F405RGTx U1
-U 1 1 611830cb
+U 1 1 611860b6
 P 16550 11650
 F 0 "U1" H 15950 13400 50 000 L CNN
@@
 $Comp
 L Device:C_Small C1
-U 1 1 611830cb
-P 15450 10550
-F 0 "C1" H 15460 10620 50 000 L CNN
-   1   15450 10550
+U 1 1 611860b6
+P 15700 10550
+F 0 "C1" H 15710 10620 50 000 L CNN
+   1   15700 10550
    1   0  0  -1
 $EndComp
 $Comp
 L Device:C_Small C2
-U 1 1 611830cb
-P 15700 10650
-F 0 "C2" H 15710 10720 50 000 L CNN
-   1   15700 10650
+U 1 1 611860b6
+P 15450 10650
+F 0 "C2" H 15460 10720 50 000 L CNN
+   1   15450 10650
    1   0  0  -1
 $EndComp
 $Comp
 L Device:D D1
-U 1 1 611830cb
-P 16550 11650
-F 0 "D1" H 16550 11750 50 000 C CNN
-   1   16550 11650
+U 1 1 611860b6
+P 17250 13600
+F 0 "D1" H 17250 13700 50 000 C CNN
+   1   17250 13600
    1   0  0  -1
 $EndComp
 $Comp
 L Device:R R1
-U 1 1 611830cb
+U 1 1 611860b6
 P 17400 11700
 F 0 "R1" V 17480 11700 50 000 C CNN
@@
 $Comp
 L 74xGxx:74LVC1G66 U2
-U 1 1 611830cb
-P 18550 13650
-F 0 "U2" H 18450 13850 50 000 C CNN
-   1   18550 13650
+U 1 1 611860b6
+P 19050 12650
+F 0 "U2" H 18950 12850 50 000 C CNN
+   1   19050 12650
    1   0  0  -1
 $EndComp
 $Comp
 L Device:R R2
-U 1 1 611830cb
-P 17800 13800
-F 0 "R2" V 17880 13800 50 000 C CNN
-   1   17800 13800
+U 1 1 611860b6
+P 18650 12800
+F 0 "R2" V 18730 12800 50 000 C CNN
+   1   18650 12800
    1   0  0  -1
 $EndComp
 $Comp
 L Device:R R3
-U 1 1 611830cb
-P 18950 13800
-F 0 "R3" V 19030 13800 50 000 C CNN
-   1   18950 13800
+U 1 1 611860b6
+P 19450 12800
+F 0 "R3" V 19530 12800 50 000 C CNN
+   1   19450 12800
    1   0  0  -1
 $EndComp
 $Comp
 L Device:C C3
-U 1 1 611830cb
-P 18550 13250
-F 0 "C3" H 18575 13350 50 000 L CNN
-   1   18550 13250
+U 1 1 611860b6
+P 19050 12650
+F 0 "C3" H 19075 12750 50 000 L CNN
+   1   19050 12650
    1   0  0  -1
 $EndComp
 $Comp
 L Device:D D2
-U 1 1 611830cb
-P 18100 13800
-F 0 "D2" H 18100 13900 50 000 C CNN
-   1   18100 13800
+U 1 1 611860b6
+P 18350 12800
+F 0 "D2" H 18350 12900 50 000 C CNN
+   1   18350 12800
    1   0  0  -1
 $EndComp
 $Comp
 L Device:R R4
-U 1 1 611830cb
-P 18550 13650
-F 0 "R4" V 18630 13650 50 000 C CNN
-   1   18550 13650
+U 1 1 611860b6
+P 19050 12650
+F 0 "R4" V 19130 12650 50 000 C CNN
+   1   19050 12650
    1   0  0  -1
 $EndComp
 Wire Wire Line
-	18300 13800 18250 13800
+	17400 11850 17100 13600
 Wire Wire Line
-	17400 11850 16400 11650
-Wire Wire Line
-	18300 13650 17800 13650
-Wire Wire Line
-	18800 13650 18950 13650
-Wire Wire Line
-	15850 10550 15700 10550
-Wire Wire Line
-	18550 13800 17950 13800
-Wire Wire Line
-	15850 10450 15450 10450
+	15850 10450 15700 10450
 Wire Wire Line
 	17250 11550 17400 11550
+Wire Wire Line
+	18800 12650 18650 12650
+Wire Wire Line
+	19300 12650 19450 12650
+Wire Wire Line
+	18800 12800 18500 12800
+Wire Wire Line
+	15850 10550 15450 10550
+Wire Wire Line
+	19050 12800 18200 12800
+Wire Notes Line
+	15350 10650 15350 13700
+Wire Notes Line
+	15350 13700 17500 13700
+Wire Notes Line
+	17500 13700 17500 10650
+Wire Notes Line
+	17500 10650 15350 10650
+Wire Notes Line
+	16550 11650 16550 12950
+Wire Notes Line
+	16550 12950 19550 12950
+Wire Notes Line
+	19550 12950 19550 11650
+Wire Notes Line
+	19550 11650 16550 11650
 $EndSCHEMATC

Commit message: Note rectangles drawing correctly
Changed lines of the file:
@@
 $Comp
 L MCU_ST_STM32F4:STM32F405RGTx U1
-U 1 1 611860b6
+U 1 1 61188f23
 P 16550 11650
 F 0 "U1" H 15950 13400 50 000 L CNN
@@
 $Comp
 L Device:C_Small C1
-U 1 1 611860b6
+U 1 1 61188f23
 P 15700 10550
 F 0 "C1" H 15710 10620 50 000 L CNN
@@
 $Comp
 L Device:C_Small C2
-U 1 1 611860b6
+U 1 1 61188f23
 P 15450 10650
 F 0 "C2" H 15460 10720 50 000 L CNN
@@
 $Comp
 L Device:D D1
-U 1 1 611860b6
+U 1 1 61188f23
 P 17250 13600
 F 0 "D1" H 17250 13700 50 000 C CNN
@@
 $Comp
 L Device:R R1
-U 1 1 611860b6
+U 1 1 61188f23
 P 17400 11700
 F 0 "R1" V 17480 11700 50 000 C CNN
@@
 $Comp
 L 74xGxx:74LVC1G66 U2
-U 1 1 611860b6
+U 1 1 61188f23
 P 19050 12650
 F 0 "U2" H 18950 12850 50 000 C CNN
@@
 $Comp
 L Device:R R2
-U 1 1 611860b6
+U 1 1 61188f23
 P 18650 12800
 F 0 "R2" V 18730 12800 50 000 C CNN
@@
 $Comp
 L Device:R R3
-U 1 1 611860b6
+U 1 1 61188f23
 P 19450 12800
 F 0 "R3" V 19530 12800 50 000 C CNN
@@
 $Comp
 L Device:C C3
-U 1 1 611860b6
+U 1 1 61188f23
 P 19050 12650
 F 0 "C3" H 19075 12750 50 000 L CNN
@@
 $Comp
 L Device:D D2
-U 1 1 611860b6
+U 1 1 61188f23
 P 18350 12800
 F 0 "D2" H 18350 12900 50 000 C CNN
@@
 $Comp
 L Device:R R4
-U 1 1 611860b6
+U 1 1 61188f23
 P 19050 12650
 F 0 "R4" V 19130 12650 50 000 C CNN
@@
    1   0  0  -1
 $EndComp
-Wire Wire Line
-	17400 11850 17100 13600
 Wire Wire Line
 	15850 10450 15700 10450
@@
 	19300 12650 19450 12650
 Wire Wire Line
+	15850 10550 15450 10550
+Wire Wire Line
 	18800 12800 18500 12800
 Wire Wire Line
-	15850 10550 15450 10550
+	17400 11850 17100 13600
 Wire Wire Line
 	19050 12800 18200 12800
 Wire Notes Line
-	15350 10650 15350 13700
+	15350 9850 15350 13700
 Wire Notes Line
 	15350 13700 17500 13700
 Wire Notes Line
-	17500 13700 17500 10650
+	17500 13700 17500 9850
 Wire Notes Line
-	17500 10650 15350 10650
+	17500 9850 15350 9850
 Wire Notes Line
-	16550 11650 16550 12950
+	18200 12500 18200 12950
 Wire Notes Line
-	16550 12950 19550 12950
+	18200 12950 19550 12950
 Wire Notes Line
-	19550 12950 19550 11650
+	19550 12950 19550 12500
 Wire Notes Line
-	19550 11650 16550 11650
+	19550 12500 18200 12500
 $EndSCHEMATC

Commit message: Cleaned up a bit
Parts:
- removed C3: (no value), symbol Device:C
- removed D2: (no value), symbol Device:D
- removed R2, R3, R4: (no value), symbol Device:R
- removed U2: (no value), symbol 74xGxx:74LVC1G66
Connections:
- wire segments 8 -> 4
Other:
- note added: "stm32f405r0"
Changed lines of the file:
@@
 encoding utf-8
 Sheet 1 1
-Title "STM32 SKiDL"
-Date "2021-08-09"
+Title "Default"
+Date "2021-8-15"
 Rev "v0.1"
 Comp ""
@@
 $Comp
 L MCU_ST_STM32F4:STM32F405RGTx U1
-U 1 1 61188f23
+U 1 1 61199df8
 P 16550 11650
 F 0 "U1" H 15950 13400 50 000 L CNN
@@
 $Comp
 L Device:C_Small C1
-U 1 1 61188f23
-P 15700 10550
-F 0 "C1" H 15710 10620 50 000 L CNN
-   1   15700 10550
+U 1 1 61199df8
+P 15450 10550
+F 0 "C1" H 15460 10620 50 000 L CNN
+   1   15450 10550
    1   0  0  -1
 $EndComp
 $Comp
 L Device:C_Small C2
-U 1 1 61188f23
-P 15450 10650
-F 0 "C2" H 15460 10720 50 000 L CNN
-   1   15450 10650
+U 1 1 61199df8
+P 15700 10650
+F 0 "C2" H 15710 10720 50 000 L CNN
+   1   15700 10650
    1   0  0  -1
 $EndComp
 $Comp
 L Device:D D1
-U 1 1 61188f23
+U 1 1 61199df8
 P 17250 13600
 F 0 "D1" H 17250 13700 50 000 C CNN
@@
 $Comp
 L Device:R R1
-U 1 1 61188f23
+U 1 1 61199df8
 P 17400 11700
 F 0 "R1" V 17480 11700 50 000 C CNN
@@
    1   0  0  -1
 $EndComp
-$Comp
-L 74xGxx:74LVC1G66 U2
-U 1 1 61188f23
-P 19050 12650
-F 0 "U2" H 18950 12850 50 000 C CNN
-   1   19050 12650
-   1   0  0  -1
-$EndComp
-$Comp
-L Device:R R2
-U 1 1 61188f23
-P 18650 12800
-F 0 "R2" V 18730 12800 50 000 C CNN
-   1   18650 12800
-   1   0  0  -1
-$EndComp
-$Comp
-L Device:R R3
-U 1 1 61188f23
-P 19450 12800
-F 0 "R3" V 19530 12800 50 000 C CNN
-   1   19450 12800
-   1   0  0  -1
-$EndComp
-$Comp
-L Device:C C3
-U 1 1 61188f23
-P 19050 12650
-F 0 "C3" H 19075 12750 50 000 L CNN
-   1   19050 12650
-   1   0  0  -1
-$EndComp
-$Comp
-L Device:D D2
-U 1 1 61188f23
-P 18350 12800
-F 0 "D2" H 18350 12900 50 000 C CNN
-   1   18350 12800
-   1   0  0  -1
-$EndComp
-$Comp
-L Device:R R4
-U 1 1 61188f23
-P 19050 12650
-F 0 "R4" V 19130 12650 50 000 C CNN
-   1   19050 12650
-   1   0  0  -1
-$EndComp
-Wire Wire Line
-	15850 10450 15700 10450
-Wire Wire Line
-	17250 11550 17400 11550
-Wire Wire Line
-	18800 12650 18650 12650
-Wire Wire Line
-	19300 12650 19450 12650
-Wire Wire Line
-	15850 10550 15450 10550
-Wire Wire Line
-	18800 12800 18500 12800
 Wire Wire Line
 	17400 11850 17100 13600
 Wire Wire Line
-	19050 12800 18200 12800
+	15850 10550 15700 10550
+Wire Wire Line
+	15850 10450 15450 10450
+Wire Wire Line
+	17250 11550 17400 11550
+Text Notes 15837 9650 0    100  ~ 20
+stm32f405r0
 Wire Notes Line
-	15350 9850 15350 13700
+	15250 9450 15250 13800
 Wire Notes Line
-	15350 13700 17500 13700
+	15250 13800 17600 13800
 Wire Notes Line
-	17500 13700 17500 9850
+	17600 13800 17600 9450
 Wire Notes Line
-	17500 9850 15350 9850
-Wire Notes Line
-	18200 12500 18200 12950
-Wire Notes Line
-	18200 12950 19550 12950
-Wire Notes Line
-	19550 12950 19550 12500
-Wire Notes Line
-	19550 12500 18200 12500
+	17600 9450 15250 9450
 $EndSCHEMATC
