File: examples/stm32_usb_buck/stm32/stm32.sch (KiCad schematic (older format))
At the start: 5 parts

Commit message: Adding hierarchical sheet to main sheet
Changed lines of the file:
@@
 Comment4 ""
 $EndDescr
+$Sheet
+S 5000 5000 1000 2000
+U 6119a4e5
+F0 "top.stm32f405r0" 100
+F1 "top.stm32f405r0.sch" 100
+$EndSheet
 $Comp
 L MCU_ST_STM32F4:STM32F405RGTx U1
-U 1 1 61199df8
+U 1 1 6119a4e5
 P 16550 11650
 F 0 "U1" H 15950 13400 50 000 L CNN
@@
 $Comp
 L Device:C_Small C1
-U 1 1 61199df8
-P 15450 10550
-F 0 "C1" H 15460 10620 50 000 L CNN
-   1   15450 10550
+U 1 1 6119a4e5
+P 15700 10550
+F 0 "C1" H 15710 10620 50 000 L CNN
+   1   15700 10550
    1   0  0  -1
 $EndComp
 $Comp
 L Device:C_Small C2
-U 1 1 61199df8
-P 15700 10650
-F 0 "C2" H 15710 10720 50 000 L CNN
-   1   15700 10650
+U 1 1 6119a4e5
+P 15450 10650
+F 0 "C2" H 15460 10720 50 000 L CNN
+   1   15450 10650
    1   0  0  -1
 $EndComp
 $Comp
 L Device:D D1
-U 1 1 61199df8
+U 1 1 6119a4e5
 P 17250 13600
 F 0 "D1" H 17250 13700 50 000 C CNN
@@
 $Comp
 L Device:R R1
-U 1 1 61199df8
+U 1 1 6119a4e5
 P 17400 11700
 F 0 "R1" V 17480 11700 50 000 C CNN
@@
 	17400 11850 17100 13600
 Wire Wire Line
-	15850 10550 15700 10550
+	15850 10450 15700 10450
 Wire Wire Line
-	15850 10450 15450 10450
+	15850 10550 15450 10550
 Wire Wire Line
 	17250 11550 17400 11550
